File: Shield_Pins.kicad_pcb (KiCad board)
At the start: 2 copper layers, 76 x 38.3 mm, 9 parts, among them J1 Conn_01x04_Male, J2 Conn_01x06_Male, J3 Conn_01x06_Male, J4 Conn_01x04_Male, J5 Conn_01x01_Male, J6 Conn_01x06_Male, J7 Conn_01x15_Male, J8 Conn_01x15_Male, J9 Conn_01x02_Male

Commit message: Init Push
Parts:
- added C1: 0.1uF, Capacitor_SMD:C_0603_1608Metric_Pad1.08x0.95mm_HandSolder, F.Cu at (113.2, 85.8)
- added C2: 22pF, Capacitor_SMD:C_0603_1608Metric_Pad1.08x0.95mm_HandSolder, F.Cu at (131.8, 80.5)
- added C3: 22pF, Capacitor_SMD:C_0603_1608Metric_Pad1.08x0.95mm_HandSolder, F.Cu at (121.9, 80.4)
- added C4: 100pF, Capacitor_SMD:C_0603_1608Metric_Pad1.08x0.95mm_HandSolder, F.Cu at (113.2, 89.8)
- added C5: 0.1uF, Capacitor_SMD:C_0603_1608Metric_Pad1.08x0.95mm_HandSolder, F.Cu at (143.9, 87.2)
- added C6: 100nF, Capacitor_SMD:C_0603_1608Metric_Pad1.08x0.95mm_HandSolder, B.Cu at (116.5, 76.5)
- added C7: 100nF, Capacitor_SMD:C_0603_1608Metric_Pad1.08x0.95mm_HandSolder, B.Cu at (97.1, 74.5)
- added CIN1: 100nF, Capacitor_SMD:C_0603_1608Metric_Pad1.08x0.95mm_HandSolder, B.Cu at (114.5, 76.5)
- added COUT1: 10uF, Capacitor_SMD:C_0603_1608Metric_Pad1.08x0.95mm_HandSolder, B.Cu at (118.5, 76.5)
- added D1: 3.3V 500mW, Diode_SMD:D_SOD-123, F.Cu at (112.5, 83.5)
- added D2: LED, LED_SMD:LED_0603_1608Metric_Pad1.05x0.95mm_HandSolder, F.Cu at (107.4, 99.9)
- added D3: LED, LED_SMD:LED_0603_1608Metric_Pad1.05x0.95mm_HandSolder, F.Cu at (107.5, 95.8)
- added D4: LED, LED_SMD:LED_0603_1608Metric_Pad1.05x0.95mm_HandSolder, F.Cu at (107.5, 93.8)
- added D5: LED, LED_SMD:LED_0603_1608Metric_Pad1.05x0.95mm_HandSolder, F.Cu at (107.5, 97.9)
- added D7: BAT165AX, Diode_SMD:D_SOD-323_HandSoldering, F.Cu at (107.7, 102.5)
- added D8: BAT165AX, Diode_SMD:D_SOD-323_HandSoldering, B.Cu at (102.7, 73.6)
- added F1: 1.5A Fuse, Fuse:Fuse_0603_1608Metric_Pad1.05x0.95mm_HandSolder, F.Cu at (113.8, 102.5)
- added FB1: 120R, Inductor_SMD:L_0603_1608Metric_Pad1.05x0.95mm_HandSolder, B.Cu at (97.1, 72.4)
- added G***: LOGO, CANBusShield:SoCET_logo, F.Cu at (143.0, 96.0)
- added J11: Screw_Terminal_01x02, TerminalBlock:TerminalBlock_bornier-2_P5.08mm, F.Cu at (141.7, 75.0)
- added J12: DB9_Male, Connector_Dsub:DSUB-9_Male_Horizontal_P2.77x2.84mm_EdgePinOffset9.90mm_Housed_MountingHolesOffset11.32mm, F.Cu at (102.5, 87.0)
- added R1: 6.3kR, Resistor_SMD:R_0603_1608Metric_Pad0.98x0.95mm_HandSolder, F.Cu at (113.2, 87.8)
- added R2: 1kR, Resistor_SMD:R_0603_1608Metric_Pad0.98x0.95mm_HandSolder, F.Cu at (113.2, 91.8)
- added R3: 100R, Resistor_SMD:R_0603_1608Metric_Pad0.98x0.95mm_HandSolder, F.Cu at (113.2, 99.9)
- added R4: 100R, Resistor_SMD:R_0603_1608Metric_Pad0.98x0.95mm_HandSolder, F.Cu at (113.2, 95.8)
- added R5: 100R, Resistor_SMD:R_0603_1608Metric_Pad0.98x0.95mm_HandSolder, F.Cu at (113.2, 93.8)
- added R6: 100R, Resistor_SMD:R_0603_1608Metric_Pad0.98x0.95mm_HandSolder, F.Cu at (113.2, 97.9)
- added SW1: SW_SPDT, CANBusShield:09.03290.01 switch, F.Cu at (113.8, 106.0)
- added U1: MCP2515-xSO, Package_SO:SOIC-18W_7.5x11.6mm_P1.27mm, F.Cu at (124.8, 88.9)
- added U2: MCP2551-I-SN, Package_SO:SOIC-8_3.9x4.9mm_P1.27mm, F.Cu at (139.8, 85.2)
- added U3: LD1117S50TR_SOT223, Package_TO_SOT_SMD:SOT-223-3_TabPin2, B.Cu at (108.6, 75.2)
- added Y1: 8MHz Crystal, Crystal:Crystal_SMD_HC49-SD, F.Cu at (126.7, 76.6)
Routing:
- net +5V: track 0.00 -> 163.0 mm, vias 0 -> 5
- net CANL: track 0.00 -> 65.7 mm, vias 0 -> 1
- net CANH: track 0.00 -> 65.6 mm, vias 0 -> 1
- net IO20: track 0.00 -> 55.9 mm, vias 0 -> 1
- net IO11: track 0.00 -> 53.5 mm, vias 0 -> 1
- net RXCAN: track 0.00 -> 46.5 mm, vias 0 -> 2
- net TXCAN: track 0.00 -> 46.5 mm, vias 0 -> 2
- net IO8: track 0.00 -> 45.6 mm
- net IO19: track 0.00 -> 44.3 mm, vias 0 -> 1
- net IO18: track 0.00 -> 44.3 mm, vias 0 -> 1
- net IO9: track 0.00 -> 43.6 mm
- net IO10: track 0.00 -> 41.6 mm
- net +3.3V: track 0.00 -> 39.1 mm
- net 12V_OBD: track 0.00 -> 35.3 mm, vias 0 -> 3
- net IO17: track 0.00 -> 25.6 mm
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- added copper zone on F.Cu, net 12V_OBD_IN
- added copper zone on B.Cu, net GND
- added copper zone on F.Cu, net GND

Commit message: Complete board (1)
Parts:
- added C8: 4.7nF, Capacitor_SMD:C_0603_1608Metric_Pad1.08x0.95mm_HandSolder, F.Cu at (150.8, 76.6)
- added D6: LED, LED_SMD:LED_0603_1608Metric_Pad1.05x0.95mm_HandSolder, F.Cu at (107.5, 100.0)
- added JP1: SolderJumper_2_Open, Connector_PinHeader_2.00mm:PinHeader_1x02_P2.00mm_Vertical, F.Cu at (147.0, 80.6)
- added Q1: NPN 15V 0.7A, Package_TO_SOT_SMD:SC-59_Handsoldering, F.Cu at (107.7, 87.8)
- added Q2: NPN 15V 0.7A, Package_TO_SOT_SMD:SC-59_Handsoldering, B.Cu at (108.3, 94.8)
- added Q3: NPN 15V 0.7A, Package_TO_SOT_SMD:SC-59_Handsoldering, B.Cu at (120.3, 101.2)
- added R7: 560R, Resistor_SMD:R_0603_1608Metric_Pad0.98x0.95mm_HandSolder, F.Cu at (113.3, 100.0)
- added R8: 60R, Resistor_SMD:R_0603_1608Metric_Pad0.98x0.95mm_HandSolder, F.Cu at (150.8, 78.6)
- added R9: 60R, Resistor_SMD:R_0603_1608Metric_Pad0.98x0.95mm_HandSolder, F.Cu at (150.8, 80.6)
- R3, R4, R5, R6: value 100R -> 150R
- moved C3 10.7 mm to (129.8, 73.2)
- moved C2 5.56 mm to (129.8, 75.2)
- moved D3 4.00 mm to (107.5, 91.8)
- moved R4 4.00 mm to (113.3, 91.8), turned to 0 degrees
- moved Y1 2.90 mm to (125.2, 79.2)
- moved G*** 2.38 mm to (143.2, 93.6)
- moved R1 2.03 mm to (113.3, 85.8)
- moved D1 2.00 mm to (112.7, 81.5)
- moved D5 2.00 mm to (107.6, 95.9)
- moved D2 2.00 mm to (107.5, 97.9)
- moved R3 2.00 mm to (113.3, 97.9)
- moved R6 2.00 mm to (113.3, 95.9)
- moved C4 2.00 mm to (113.3, 87.8)
- moved C1 2.00 mm to (113.3, 83.8)
- moved R2 2.00 mm to (113.3, 89.8)
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Connections:
- D3 pad 1: GND -> Net-(D3-Pad1)
- D4 pad 1: GND -> Net-(D4-Pad1)
- D5 pad 1: GND -> Net-(D5-Pad1)
- R4 pad 1: RXCAN -> Net-(D3-Pad2)
- R4 pad 2: Net-(D3-Pad2) -> +5V
- R5 pad 1: TXCAN -> Net-(D4-Pad2)
- R5 pad 2: Net-(D4-Pad2) -> +5V
- R6 pad 1: IO20 -> +5V
Routing:
- net Net-(D5-Pad1): track 0.00 -> 21.0 mm, vias 0 -> 1
- net CANL: track 65.7 -> 84.9 mm
- net CANH: track 65.6 -> 84.8 mm
- net OSC1: track 8.23 -> 17.7 mm
- net 12V_OBD: track 35.3 -> 41.4 mm
- net +5V: track 163.0 -> 168.6 mm
- net Net-(D4-Pad1): track 0.00 -> 5.30 mm, vias 0 -> 1
- net GND: track 3.95 -> 9.00 mm, vias 68 -> 49
- net IO20: track 55.9 -> 51.1 mm, vias 1 -> 2
- net TXCAN: track 46.5 -> 50.9 mm, vias 2 -> 1
- net Net-(R8-Pad2): track 0.00 -> 4.02 mm
- net Net-(D6-Pad2): track 0.00 -> 4.01 mm
- net RXCAN: track 46.5 -> 42.9 mm
- net Net-(D3-Pad1): track 0.00 -> 3.25 mm
- net ~{CAN_RST}: track 19.4 -> 18.5 mm
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Other:
- board text added: "AFT-x06 CAN-BUS Shield Minh Nguyen Rauf Emre Erkiletlioglu"

Commit message: Complete board (2)
Parts:
- C6, C7, CIN1: footprint Capacitor_SMD:C_0603_1608Metric_Pad1.08x0.95mm_HandSolder -> Capacitor_SMD:C_0805_2012Metric_Pad1.18x1.45mm_HandSolder
- D1: footprint Diode_SMD:D_SOD-123 -> Diode_SMD:D_SOD-323_HandSoldering
- R7: value 560R -> 634R
- moved COUT1 0.89 mm to (119.4, 76.7)
- moved C6 0.79 mm to (117.3, 76.7)
- moved D1 0.65 mm to (113.3, 81.5)
- moved CIN1 0.37 mm to (114.8, 76.7)
- moved C7 0.17 mm to (97.3, 74.5)
Routing:
- net 5V_OBD: track 17.3 -> 18.3 mm
- net Net-(C4-Pad1): track 11.3 -> 12.3 mm
