File: Shield_Pins.kicad_pcb (KiCad board)
At the start: 2 copper layers, 76 x 38.3 mm, 9 parts, among them J1 Conn_01x04_Male, J2 Conn_01x06_Male, J3 Conn_01x06_Male, J4 Conn_01x04_Male, J5 Conn_01x01_Male, J6 Conn_01x06_Male, J7 Conn_01x15_Male, J8 Conn_01x15_Male, J9 Conn_01x02_Male

Commit message: next commit
Parts:
- added C1: 1uF, Capacitor_SMD:C_0805_2012Metric, F.Cu at (144.1, 92.1)
- added C2: 100 nF, Capacitor_SMD:C_0805_2012Metric, F.Cu at (129.8, 93.8)
- added C3: 1uF, Capacitor_SMD:C_0805_2012Metric, F.Cu at (144.2, 88.5)
- added C4: 0.1uF, Capacitor_SMD:C_0805_2012Metric, F.Cu at (144.2, 85.5)
- added C5: 1uF, Capacitor_SMD:C_0805_2012Metric, F.Cu at (134.3, 93.8)
- added C6: 100 nF, Capacitor_SMD:C_0805_2012Metric, F.Cu at (139.7, 92.1)
- added U1: ADXL343, Package_LGA:LGA-14_3x5mm_P0.8mm_LayoutBorder1x6y, F.Cu at (139.7, 87.3)
- added U2: AZ1117, Package_TO_SOT_SMD:SOT-223-3_TabPin2, F.Cu at (132.5, 88.1)

Commit message: pcb initial
Parts:
- moved C1 15.4 mm to (129.9, 97.8)
- moved C4 8.67 mm to (135.6, 85.5), turned to 180 degrees
- moved C2 7.82 mm to (129.8, 101.6)
- moved C5 6.92 mm to (140.3, 97.2)
- moved U1 6.61 mm to (146.3, 86.6)
- moved C3 4.87 mm to (139.4, 88.3), turned to 180 degrees
- moved U2 3.57 mm to (132.1, 91.7)
Routing:
- net +3V3: track 0.00 -> 19.2 mm
- net +3.3V: track 0.00 -> 15.3 mm
- added copper zone on F.Cu, net +5V
- added copper zone on B.Cu, net GND
- added copper zone on F.Cu, net GND
Changed lines of the file:
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@@
   (net 52 "IO{SCK}")
   (footprint "Capacitor_SMD:C_0805_2012Metric" (layer "F.Cu")
-    (at 129.845 93.775)
+    (at 129.845 101.6)
     (descr "Capacitor SMD 0805 (2012 Metric), square (rectangular) end terminal, IPC_7351 nominal, (Body size source: IPC-SM-782 page 76, https://www.pcb-3d.com/wordpress/wp-content/uploads/ipc-sm-782a_amendment_1_and_2.pdf, https://docs.google.com/spreadsheets/d/1BsfQQcO9C6DZCsRaXUlFlo91Tg2WpOkGARC1WS5S8t0/edit?usp=sharing), generated with kicad-footprint-generator")
     (tags "capacitor")
@@
   )
   (footprint "Package_TO_SOT_SMD:SOT-223-3_TabPin2" (layer "F.Cu")
-    (at 132.545 88.145)
+    (at 132.055 91.68)
     (descr "module CMS SOT223 4 pins")
     (tags "CMS SOT")
@@
   )
   (footprint "Package_LGA:LGA-14_3x5mm_P0.8mm_LayoutBorder1x6y" (layer "F.Cu")
-    (at 139.745 87.295)
+    (at 146.32 86.595)
     (descr "LGA, 14 Pin (http://www.st.com/resource/en/datasheet/lsm303dlhc.pdf), generated with kicad-footprint-generator ipc_noLead_generator.py")
     (tags "LGA NoLead")
@@
   )
   (footprint "Capacitor_SMD:C_0805_2012Metric" (layer "F.Cu")
-    (at 134.295 93.775)
+    (at 140.335 97.155)
     (descr "Capacitor SMD 0805 (2012 Metric), square (rectangular) end terminal, IPC_7351 nominal, (Body size source: IPC-SM-782 page 76, https://www.pcb-3d.com/wordpress/wp-content/uploads/ipc-sm-782a_amendment_1_and_2.pdf, https://docs.google.com/spreadsheets/d/1BsfQQcO9C6DZCsRaXUlFlo91Tg2WpOkGARC1WS5S8t0/edit?usp=sharing), generated with kicad-footprint-generator")
     (tags "capacitor")
@@
   )
   (footprint "Capacitor_SMD:C_0805_2012Metric" (layer "F.Cu")
-    (at 144.245 88.535)
+    (at 139.385 88.265 180)
     (descr "Capacitor SMD 0805 (2012 Metric), square (rectangular) end terminal, IPC_7351 nominal, (Body size source: IPC-SM-782 page 76, https://www.pcb-3d.com/wordpress/wp-content/uploads/ipc-sm-782a_amendment_1_and_2.pdf, https://docs.google.com/spreadsheets/d/1BsfQQcO9C6DZCsRaXUlFlo91Tg2WpOkGARC1WS5S8t0/edit?usp=sharing), generated with kicad-footprint-generator")
     (tags "capacitor")
@@
     (fp_line (start -1 -0.625) (end 1 -0.625) (layer "F.Fab") (width 0.1))
     (fp_line (start 1 0.625) (end -1 0.625) (layer "F.Fab") (width 0.1))
-    (pad "1" smd roundrect locked (at -0.95 0) (size 1 1.45) (layers "F.Cu" "F.Paste" "F.Mask") (roundrect_rratio 0.25)
+    (pad "1" smd roundrect locked (at -0.95 0 180) (size 1 1.45) (layers "F.Cu" "F.Paste" "F.Mask") (roundrect_rratio 0.25)
       (net 43 "+3V3") (pintype "passive"))
-    (pad "2" smd roundrect locked (at 0.95 0) (size 1 1.45) (layers "F.Cu" "F.Paste" "F.Mask") (roundrect_rratio 0.25)
+    (pad "2" smd roundrect locked (at 0.95 0 180) (size 1 1.45) (layers "F.Cu" "F.Paste" "F.Mask") (roundrect_rratio 0.25)
       (net 4 "GND") (pintype "passive"))
     (model "${KICAD6_3DMODEL_DIR}/Capacitor_SMD.3dshapes/C_0805_2012Metric.wrl"
@@
   )
   (footprint "Capacitor_SMD:C_0805_2012Metric" (layer "F.Cu")
-    (at 144.145 92.075)
+    (at 129.855 97.79)
     (descr "Capacitor SMD 0805 (2012 Metric), square (rectangular) end terminal, IPC_7351 nominal, (Body size source: IPC-SM-782 page 76, https://www.pcb-3d.com/wordpress/wp-content/uploads/ipc-sm-782a_amendment_1_and_2.pdf, https://docs.google.com/spreadsheets/d/1BsfQQcO9C6DZCsRaXUlFlo91Tg2WpOkGARC1WS5S8t0/edit?usp=sharing), generated with kicad-footprint-generator")
     (tags "capacitor")
@@
   )
   (footprint "Capacitor_SMD:C_0805_2012Metric" (layer "F.Cu")
-    (at 144.245 85.525)
+    (at 135.575 85.525 180)
     (descr "Capacitor SMD 0805 (2012 Metric), square (rectangular) end terminal, IPC_7351 nominal, (Body size source: IPC-SM-782 page 76, https://www.pcb-3d.com/wordpress/wp-content/uploads/ipc-sm-782a_amendment_1_and_2.pdf, https://docs.google.com/spreadsheets/d/1BsfQQcO9C6DZCsRaXUlFlo91Tg2WpOkGARC1WS5S8t0/edit?usp=sharing), generated with kicad-footprint-generator")
     (tags "capacitor")
@@
     (fp_line (start -1 -0.625) (end 1 -0.625) (layer "F.Fab") (width 0.1))
     (fp_line (start 1 0.625) (end -1 0.625) (layer "F.Fab") (width 0.1))
-    (pad "1" smd roundrect locked (at -0.95 0) (size 1 1.45) (layers "F.Cu" "F.Paste" "F.Mask") (roundrect_rratio 0.25)
+    (pad "1" smd roundrect locked (at -0.95 0 180) (size 1 1.45) (layers "F.Cu" "F.Paste" "F.Mask") (roundrect_rratio 0.25)
       (net 43 "+3V3") (pintype "passive"))
-    (pad "2" smd roundrect locked (at 0.95 0) (size 1 1.45) (layers "F.Cu" "F.Paste" "F.Mask") (roundrect_rratio 0.25)
+    (pad "2" smd roundrect locked (at 0.95 0 180) (size 1 1.45) (layers "F.Cu" "F.Paste" "F.Mask") (roundrect_rratio 0.25)
       (net 4 "GND") (pintype "passive"))
     (model "${KICAD6_3DMODEL_DIR}/Capacitor_SMD.3dshapes/C_0805_2012Metric.wrl"
@@
     (style (thickness 0.1) (arrow_length 1.27) (text_position_mode 0) (extension_height 0.58642) (extension_offset 0.5) keep_text_aligned)
   )
+  (segment (start 138.35 91.68) (end 138.745 92.075) (width 0.25) (layer "F.Cu") (net 9))
+  (segment (start 135.205 91.68) (end 128.905 91.68) (width 0.25) (layer "F.Cu") (net 9))
+  (segment (start 139.385 97.155) (end 139.385 92.715) (width 0.25) (layer "F.Cu") (net 9))
+  (segment (start 139.385 92.715) (end 138.745 92.075) (width 0.25) (layer "F.Cu") (net 9))
+  (segment (start 135.205 91.68) (end 138.35 91.68) (width 0.25) (layer "F.Cu") (net 9))
   (segment (start 160.15 100.6) (end 160.175 100.575) (width 0.25) (layer "F.Cu") (net 16))
+  (segment (start 136.755 85.295) (end 136.525 85.525) (width 0.25) (layer "F.Cu") (net 43))
+  (segment (start 137.595 85.725) (end 136.525 85.725) (width 0.25) (layer "F.Cu") (net 43))
+  (segment (start 138.925 84.595) (end 145.32 84.595) (width 0.25) (layer "F.Cu") (net 43))
+  (segment (start 140.335 88.265) (end 140.665 88.595) (width 0.25) (layer "F.Cu") (net 43))
+  (segment (start 138.225 85.295) (end 136.755 85.295) (width 0.25) (layer "F.Cu") (net 43))
+  (segment (start 140.335 88.465) (end 137.595 85.725) (width 0.25) (layer "F.Cu") (net 43))
+  (segment (start 140.665 88.595) (end 145.32 88.595) (width 0.25) (layer "F.Cu") (net 43))
+  (segment (start 138.225 85.295) (end 138.925 84.595) (width 0.25) (layer "F.Cu") (net 43))
+  (zone (net 1) (net_name "+5V") (layer "F.Cu") (hatch edge 0.508)
+    (priority 1)
+    (connect_pads (clearance 0.508))
+    (min_thickness 0.254) (filled_areas_thickness no)
+    (fill yes (thermal_gap 0.508) (thermal_bridge_width 0.508))
+    (polygon
+      (pts
+        (xy 129.54 107.95)
+        (xy 127.635 107.95)
+        (xy 127.635 92.71)
+        (xy 129.54 92.71)
+      )
+    )
+  )
+  (zone (net 4) (net_name "GND") (layers F&B.Cu) (hatch edge 0.508)
+    (connect_pads (clearance 0.508))
+    (min_thickness 0.254) (filled_areas_thickness no)
+    (fill yes (thermal_gap 0.508) (thermal_bridge_width 0.508))
+    (polygon
+      (pts
+        (xy 165.735 109.855)
+        (xy 88.9 109.22)
+        (xy 88.9 69.85)
+        (xy 165.625 69.85)
+      )
+    )
+  )
 )

Commit message: Revised PCB and Sheet
Parts:
- added D1: LED, LED_SMD:LED_1812_4532Metric_Pad1.30x3.40mm_HandSolder, F.Cu at (114.3, 97.2)
- added R1: 200Ω, Resistor_SMD:R_0805_2012Metric, F.Cu at (121.0, 92.1)
- moved U1 4.44 mm to (150.8, 86.6)
Connections:
- C3 pad 1: +3V3 -> 3.3V
- C4 pad 1: +3V3 -> 3.3V
- C5 pad 1: +3.3V -> 3.3V
- C6 pad 1: +3.3V -> 3.3V
- J3 pad 1: +3.3V -> 3.3V
- J6 pad 3: +3.3V -> 3.3V
- J6 pad 4: +3.3V -> 3.3V
- U1 pad 1: +3V3 -> 3.3V
- U1 pad 12: IO{SDI} -> IO.SDO
- U1 pad 13: IO{SDO} -> IO.SDI
- U1 pad 14: IO{SCK} -> IO.SCK
- U1 pad 6: +3V3 -> 3.3V
- U1 pad 7: IO{CSB} -> IO.CSB
- U1 pad 8: IO{7} -> IO7
- U2 pad 2: +3.3V -> 3.3V
Routing:
- net IO.SCK: track 0.00 -> 59.8 mm, vias 0 -> 2
- net 3.3V: track 0.00 -> 56.9 mm
- net IO.SDI: track 0.00 -> 44.7 mm
- net IO.SDO: track 0.00 -> 35.3 mm, vias 0 -> 2
- net IO.CSB: track 0.00 -> 29.1 mm
- net IO7: track 0.04 -> 20.4 mm, vias 0 -> 2
- net +3V3: track 19.2 -> 0.00 mm
- net +3.3V: track 15.3 -> 0.00 mm
- net Net-(D1-Pad2): track 0.00 -> 6.56 mm
- net GND: track 0.00 -> 3.83 mm

Commit message: Finished shield design
Parts:
- moved C2 42.9 mm to (97.0, 74.0), turned to -90 degrees
- moved C5 40.2 mm to (103.5, 81.2), turned to 180 degrees
- moved C1 38.7 mm to (99.4, 74.0), turned to -90 degrees
- moved C6 37.2 mm to (103.5, 83.4), turned to 180 degrees
- moved U1 33.6 mm to (117.6, 91.9)
- moved U2 32.0 mm to (104.4, 75.6), turned to -90 degrees
- moved C3 25.0 mm to (114.3, 87.5)
- moved C4 24.7 mm to (114.1, 97.7)
- moved R1 21.9 mm to (110.2, 73.0), turned to -90 degrees
- moved D1 20.2 mm to (112.4, 77.0), turned to 180 degrees
Routing:
- net IO.SCK: track 59.8 -> 24.4 mm, vias 2 -> 0
- net IO7: track 20.4 -> 44.4 mm
- net IO.SDI: track 44.7 -> 26.4 mm, vias 0 -> 2
- net GND: track 3.83 -> 20.8 mm, vias 0 -> 5
- net 3.3V: track 56.9 -> 41.8 mm, vias 0 -> 2
- net IO.CSB: track 29.1 -> 22.1 mm, vias 0 -> 2
- net IO.SDO: track 35.3 -> 28.8 mm
- net Net-(D1-Pad2): track 6.56 -> 3.10 mm
