File: ESP32.kicad_sch (KiCad schematic)
At the start: 6 parts, among them U1 ESP32-WROOM-32

Commit message: Revised Version
Parts:
- added C2, C3: 10uF, Capacitor_SMD:C_1206_3216Metric, symbol Device:C
- added D1: D_Schottky, Diode_SMD:D_1206_3216Metric, symbol Device:D_Schottky
- added D2, D3: LED, LED_SMD:LED_1206_3216Metric, symbol Device:LED
- added IO16-23, IO35-25: Conn_01x07_Male, Connector_PinHeader_2.00mm:PinHeader_1x07_P2.00mm_Vertical, symbol Connector:Conn_01x07_Male
- added J1: Conn_01x06_Male, Connector_PinHeader_2.00mm:PinHeader_1x06_P2.00mm_Vertical, symbol Connector:Conn_01x06_Male
- added J12: Conn_01x03_Male, Connector_PinHeader_2.00mm:PinHeader_1x03_P2.00mm_Vertical, symbol Connector:Conn_01x03_Male
- added Q1, Q2: BC807, Package_TO_SOT_SMD:SOT-23, symbol Transistor_BJT:BC807
- added R2: 10k, Resistor_SMD:R_1206_3216Metric, symbol Device:R
- added R3, R4, R5, R6: 10K, Resistor_SMD:R_1206_3216Metric, symbol Device:R
- added U1: MIC5219-2.5YM5, Package_TO_SOT_SMD:SOT-23-5, symbol Regulator_Linear:MIC5219-2.5YM5
- C1: footprint (none) -> Capacitor_SMD:C_1206_3216Metric
- C4: renamed from C2; footprint (none) -> Capacitor_SMD:C_1206_3216Metric
- C5: renamed from C3; footprint (none) -> Capacitor_SMD:C_1206_3216Metric
- R1: footprint (none) -> Resistor_SMD:R_1206_3216Metric
- SW1: renamed from SW?; footprint (none) -> Button_Switch_SMD:SW_SPST_B3U-1000P-B
- renumbered U1 to U2
Connections:
- net +3.3V: now also D1.1 (K), Q1.2 (E), Q2.2 (E), R3.2, R4.2, R6.1
- net IO.RX: now also Q2.1 (B)
- net IO.TX: now also Q1.1 (B)
- net IO 25: now reaches U2.10 (IO25)
- net IO 25: now also IO35-25.1 (Pin_1)
- net IO 26: now reaches U2.11 (IO26)
- net IO 26: now also IO35-25.2 (Pin_2)
- net IO 27: now reaches U2.12 (IO27)
- net IO 27: now also IO35-25.3 (Pin_3)
- net IO 14: now reaches U2.13 (IO14)
- net IO 14: now also J12.3 (Pin_3)
- net at U2.14 (IO12): now also R2.1
- net IO 13: now reaches U2.16 (IO13)
- net IO 13: now also J12.2 (Pin_2)
- net ESP32_SHD: now reaches U2.17 (SHD/SD2)
- net ESP32_SHD: now also J1.3 (Pin_3)
- net ESP32_SWP: now reaches U2.18 (SWP/SD3)
- net ESP32_SWP: now also J1.4 (Pin_4)
- net ESP32_SCS: now reaches U2.19 (SCS/CMD)
- net ESP32_SCS: now also J1.6 (Pin_6)
- net ESP32_SCK: now reaches U2.20 (SCK/CLK)
- net ESP32_SCK: now also J1.5 (Pin_5)
- net ESP32_SD0: now reaches U2.21 (SDO/SD0)
- net ESP32_SD0: now also J1.1 (Pin_1)
- net ESP32_SDI: now reaches U2.22 (SDI/SD1)
- net ESP32_SDI: now also J1.2 (Pin_2)
- net at U2.23 (IO15): now also R3.1
- net at U2.24 (IO2): now also R4.1
- net at U2.25 (IO0): now also R5.1
- net IO 4: now reaches U2.26 (IO4)
- net IO 4: now also J12.1 (Pin_1)
- net IO 16: now reaches U2.27 (IO16)
- net IO 16: now also IO16-23.1 (Pin_1)
- net IO 17: now reaches U2.28 (IO17)
- net IO 17: now also IO16-23.2 (Pin_2)
- net at U2.29 (IO5): now also R6.2
- net IO 18: now reaches U2.30 (IO18)
- net IO 18: now also IO16-23.3 (Pin_3)
- net IO 19: now reaches U2.31 (IO19)
- net IO 19: now also IO16-23.4 (Pin_4)
- net IO 21: now reaches U2.33 (IO21)
- net IO 21: now also IO16-23.5 (Pin_5)
- net IO 22: now reaches U2.36 (IO22)
- net IO 22: now also IO16-23.6 (Pin_6)
- net IO 23: now reaches U2.37 (IO23)
- net IO 23: now also IO16-23.7 (Pin_7)
- net IO 34: now reaches U2.6 (IO34)
- net IO 34: now also IO35-25.6 (Pin_6)
- net IO 35: now reaches U2.7 (IO35)
- net IO 35: now also IO35-25.7 (Pin_7)
- net IO 32: now reaches U2.8 (IO32)
- net IO 32: now also IO35-25.4 (Pin_4)
- net IO 33: now reaches U2.9 (IO33)
- net IO 33: now also IO35-25.5 (Pin_5)
- net GND renamed +5V
- net +5V: now also C2.2, C3.2, D2.1 (K), D3.1 (K), R2.2, R5.2, U1.1 (IN), U1.2 (GND), U1.3 (EN)
- new net: C2.1, C3.1, D1.2 (A), U1.5 (OUT)
- new net: D2.2 (A), Q1.3 (C)
- new net: D3.2 (A), Q2.3 (C)
- no-connect marks 4 -> 7
Other:
- removed sheet Power regulator
- note added: "Communication Pin TEST"
- note added: "Connector Pins"
- note added: "Power Regulator"
- moved on the sheet: C4, C5
