File: Ethernet_Shield.kicad_sch (KiCad schematic)
At the start: 31 parts, among them J10 Conn_02x15_Row_Letter_Last_Mo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, J11 Conn_02x03_Row_Letter_Last, J12 Conn_02x04_Row_Letter_Last, J13 Conn_02x03_Row_Letter_Last, J14 Conn_02x08_Row_Letter_Last, J15 RJ45, Q2 2N2219, SW1 SW_Push, U1 W5100, U2 74LVC1GU04DRL, Y1 25 MHz

Commit message: Vijay
Parts:
- removed C1: 0.1 uF, symbol Device:C
- removed D7: D, symbol Device:D
- removed E1: L78L33_SO8, Package_SO:SOIC-8_3.9x4.9mm_P1.27mm, symbol Regulator_Linear:L78L33_SO8
- removed J10: Conn_02x15_Row_Letter_Last_MountingPin, symbol Connector_Generic_MountingPin:Conn_02x15_Row_Letter_Last_MountingPin
- removed J11, J13: Conn_02x03_Row_Letter_Last, symbol Connector_Generic:Conn_02x03_Row_Letter_Last
- removed J12: Conn_02x04_Row_Letter_Last, symbol Connector_Generic:Conn_02x04_Row_Letter_Last
- removed J14: Conn_02x08_Row_Letter_Last, symbol Connector_Generic:Conn_02x08_Row_Letter_Last
- removed Q2: 2N2219, Package_TO_SOT_THT:TO-39-3, symbol Transistor_BJT:2N2219
- added C10, C11, C14, C9: 10 uF, Capacitor_SMD:CP_Elec_4x4.5, symbol Device:C_Polarized_US
- added C12: 0.01 uF, Capacitor_SMD:C_1206_3216Metric, symbol Device:C
- added C13, C6, C7: 0.1 uF, Capacitor_SMD:C_1206_3216Metric, symbol Device:C
- added C4, C5: 1 uF, Capacitor_SMD:C_1206_3216Metric, symbol Device:C
- added C8: 3.3 uF, Capacitor_SMD:CP_Elec_4x4.5, symbol Device:C_Polarized_US
- added D8: D_Schottky, Diode_SMD:D_1206_3216Metric, symbol Device:D_Schottky
- added J10: Conn_01x15_Male, Connector_PinHeader_2.54mm:PinHeader_1x15_P2.54mm_Vertical, symbol Connector:Conn_01x15_Male
- added J11, J13: Conn_01x03_Male, Connector_PinHeader_2.54mm:PinHeader_1x03_P2.54mm_Vertical, symbol Connector:Conn_01x03_Male
- added J12: Conn_01x04_Male, Connector_PinHeader_2.54mm:PinHeader_1x04_P2.54mm_Vertical, symbol Connector:Conn_01x04_Male
- added J14: Conn_01x08_Male, Connector_PinHeader_2.54mm:PinHeader_1x08_P2.54mm_Vertical, symbol Connector:Conn_01x08_Male
- added L1, L2: 1 uH, Inductor_SMD:L_1206_3216Metric, symbol Device:L
- added U3: AP2127K-3.3, Package_TO_SOT_SMD:SOT-23-5, symbol Regulator_Linear:AP2127K-3.3
- C2, C3: footprint (none) -> Capacitor_SMD:C_1206_3216Metric
- D1, D2, D3, D4, D5, D6: footprint (none) -> LED_SMD:LED_1206_3216Metric
- J15: footprint (none) -> Connector_RJ:RJ45_OST_PJ012-8P8CX_Vertical
- R1: value 1K -> 10K; footprint (none) -> Resistor_SMD:R_1206_3216Metric
- R2, R3, R4, R5, R6, R7, R8, R9: footprint (none) -> Resistor_SMD:R_1206_3216Metric
- SW1: footprint (none) -> Button_Switch_THT:SW_CW_GPTS203211B
- Y1: footprint (none) -> Crystal:Crystal_SMD_Abracon_ABM3-2Pin_5.0x3.2mm
Connections:
- net RST is gone; now on net 3V3_REG: U1.59 (~{RESET})
- net 3V3_REG: now also R1.2, C10.1, C13.1, C6.2, C7.2, D8.1 (K), L2.1; no longer U1.2 (VCC3V3A)
- net AC0: now also J13.3 (Pin_3)
- net AC1: now also J13.2 (Pin_2)
- net AC2: now also J13.1 (Pin_1)
- net ADR0: now also J10.15 (Pin_15)
- net ADR1: now also J10.14 (Pin_14)
- net ADR10: now also J10.5 (Pin_5)
- net ADR11: now also J10.4 (Pin_4)
- net ADR12: now also J10.3 (Pin_3)
- net ADR13: now also J10.2 (Pin_2)
- net ADR14: now also J10.1 (Pin_1)
- net ADR2: now also J10.13 (Pin_13)
- net ADR3: now also J10.12 (Pin_12)
- net ADR4: now also J10.11 (Pin_11)
- net ADR5: now also J10.10 (Pin_10)
- net ADR6: now also J10.9 (Pin_9)
- net ADR7: now also J10.8 (Pin_8)
- net ADR8: now also J10.7 (Pin_7)
- net ADR9: now also J10.6 (Pin_6)
- net DATA0: now also J14.8 (Pin_8)
- net DATA1: now also J14.7 (Pin_7)
- net DATA2: now also J14.6 (Pin_6)
- net DATA3: now also J14.5 (Pin_5)
- net DATA4: now also J14.4 (Pin_4)
- net DATA5: now also J14.3 (Pin_3)
- net DATA6: now also J14.2 (Pin_2)
- net DATA7: now also J14.1 (Pin_1)
- net GND: now also SW1.2, C10.2, C13.2, C4.2, C5.2, C6.1, C7.1, C8.2, C9.2, U3.2 (GND); no longer U1.10 (GNDA), U1.4 (GNDA), U1.77 (GNDA)
- net OPM0: now also J11.3 (Pin_3)
- net OPM1: now also J11.2 (Pin_2)
- net OPM2: now also J11.1 (Pin_1)
- net TEST0: now also J12.4 (Pin_4)
- net TEST1: now also J12.3 (Pin_3)
- net TEST2: now also J12.2 (Pin_2)
- net TEST3: now also J12.1 (Pin_1)
- net 1V8OUT: now reaches U1.11 (1V8_OUT), U1.15 (VCC1V8D), U1.16 (VCC1V8D), U1.33 (VCC1V8D), U1.69 (VCC1V8D)
- net 1V8OUT: now also C8.1, C9.1, L1.1; no longer U1.7 (VCC1V8A), U1.74 (VCC1V8A)
- net IO7 renamed IO8
- new net: C5.1, D8.2 (A), U3.5 (VOUT)
- new net +5V: C4.1, U3.1 (VIN), U3.3 (EN)
- new net 1V8A: C14.1, L1.2, U1.7 (VCC1V8A), U1.74 (VCC1V8A)
- new net 3V3A: C11.1, C12.2, L2.2, U1.2 (VCC3V3A)
- new net GNDA: C11.2, C12.1, C14.2, U1.10 (GNDA), U1.4 (GNDA), U1.77 (GNDA)
- no-connect marks 5 -> 4
Other:
- moved on the sheet: C2, C3, R3, SW1, Y1
