File: Shield_Pins.kicad_sch (KiCad schematic)
At the start: 38 parts, among them J10 Conn_01x01_Male, J11 Conn_01x02_Male, J12 Conn_01x01_Male, J13 Conn_01x01_Male, P1 USB_C_Plug_USB2.0, SW1 SW_DIP_x01, SW2 SW_DIP_x01, SW3 SW_Push, U1 NEO-M8Q, U2 AP2127N-3.3, U3 AP2127N-3.3, U4 74LS157, U5 74LVC1G18

Commit message: design put into new sheet and revised
Parts:
- removed AE1: W3011A, symbol Device:Antenna
- removed BT1: Battery_Cell, symbol Device:Battery_Cell
- removed C1, C2: 0.1 µF, Capacitor_SMD:C_0603_1608Metric, symbol Device:C
- removed C3, C4, C5, C6, C7: 0.1 µF, symbol Device:C
- removed D1, D5, D6: BAT165AX, Diode_SMD:D_0402_1005Metric, symbol Device:D_Schottky
- removed D2, D3, D4: LED, symbol Device:LED
- removed FB1: 120R, Inductor_SMD:L_0603_1608Metric, symbol Device:FerriteBead
- removed FL1: B39162B8813P810, Filter:Filter_1109-5_1.1x0.9mm, symbol Filter:B39162B8813P810
- removed J10, J12, J13: Conn_01x01_Male, symbol Connector:Conn_01x01_Male
- removed J11: Conn_01x02_Male, symbol Connector:Conn_01x02_Male
- removed L1, L2: 5.1 nH, symbol Device:L
- removed P1: USB_C_Plug_USB2.0, symbol Connector:USB_C_Plug_USB2.0
- removed R1: 5.1k, symbol Device:R
- removed R2, R3: 330, symbol Device:R
- removed R4: 150, symbol Device:R
- removed R5: 10k, symbol Device:R
- removed R6: 11k, symbol Device:R
- removed SW1, SW2: SW_DIP_x01, symbol Switch:SW_DIP_x01
- removed SW3: SW_Push, symbol Switch:SW_Push
- removed U1: NEO-M8Q, RF_GPS:ublox_NEO, symbol RF_GPS:NEO-M8Q
- removed U2, U3: AP2127N-3.3, Package_TO_SOT_SMD:SOT-23, symbol Regulator_Linear:AP2127N-3.3
- removed U4: 74LS157, symbol 74xx:74LS157
- removed U5: 74LVC1G18, symbol 74xGxx:74LVC1G18
Connections:
- no-connect marks 8 -> 2
Other:
- added sheet GPS_Shield (Neo_M8_GPS_Shield.kicad_sch)
- note removed: "1 to 2 Demultiplexer for Transmit"
- note removed: "2 to 1 Multiplexer"
- note removed: "3.3V I/O PINS ASSUMED"
- note removed: "Additional Pins"
- note removed: "Backup Battery"
- note removed: "GNSS Module - Ublox NEO-M8Q-01A"
- note removed: "GNSS module detects board and USB power separately."
- note removed: "High Pass Pi Filter is also viable. Inductors as suggested by SAW filter datasheet."
- note removed: "Main Board 5V to 3.3V"
- note removed: "Passive Antenna with Switch"
- note removed: "Power and Status LEDs"
- note removed: "Reset Circuit"
- note removed: "UART/I2C or SPI Switch"
- note removed: "USB 5V to 3.3V"
- note removed: "USB C Connection"
- note removed: "USB PWR Filtering - Taken from X06"
