File: Shield_Pins.kicad_sch (KiCad schematic)
At the start: 0 parts

Commit message: Initial schematic
Parts:
- added C1, C5: 1uF, Capacitor_SMD:C_0805_2012Metric, symbol Device:C
- added C2, C6: 100 nF, Capacitor_SMD:C_0805_2012Metric, symbol Device:C
- added C3: 1uF, symbol Device:C
- added C4: 0.1uF, symbol Device:C
- added U1: ADXL343, Package_LGA:LGA-14_3x5mm_P0.8mm_LayoutBorder1x6y, symbol Sensor_Motion:ADXL343
- added U2: AZ1117, Package_TO_SOT_SMD:SOT-223-3_TabPin2, symbol Regulator_Linear:AZ1117-3.3
Connections:
- new net +3.3V: C5.1, C6.1, U2.2 (VO)
- new net +3V3: C3.1, C4.1, U1.1 (Vdd_I/O), U1.6 (Vs)
- new net +5V: C1.1, C2.1, U2.3 (VI)
- new net GND: C1.2, C2.2, C3.2, C4.2, C5.2, C6.2, U1.2 (GND), U1.4 (GND), U1.5 (GND), U2.1 (GND)
- new net INT: U1.8 (INT1)

Commit message: next commit
Parts:
- C3, C4: footprint (none) -> Capacitor_SMD:C_0805_2012Metric
Connections:
- net IO{SDI}: now reaches U1.12 (SDO/ADDR)
- net IO{SDO}: now reaches U1.13 (SDA/SDI/SDIO)
- net IO{SCK}: now reaches U1.14 (SCL/SCLK)
- net IO{CSB}: now reaches U1.7 (~{CS})
- net INT renamed IO{7}
- no-connect marks 5 -> 6
Changed lines of the file:
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@@
   (no_connect (at 55.88 63.5))
   (no_connect (at 45.72 38.1))
+  (no_connect (at 63.5 53.34))
   (no_connect (at 139.7 21.59))
   (no_connect (at 139.7 26.67))
@@
     (effects (font (size 1.27 1.27) (thickness 0.254) bold) (justify left bottom))
   )
-  (global_label "INT" (shape input) (at 63.5 50.8 0) (fields_autoplaced)
+  (global_label "IO{CSB}" (shape input) (at 38.1 55.88 180) (fields_autoplaced)
+    (effects (font (size 1.27 1.27)) (justify right))
+    (property "Intersheet References" "${INTERSHEET_REFS}" (id 0) (at 28.3088 55.8006 0)
+      (effects (font (size 1.27 1.27)) (justify right) hide)
+    )
+  )
+  (global_label "IO{7}" (shape input) (at 63.5 50.8 0) (fields_autoplaced)
     (effects (font (size 1.27 1.27)) (justify left))
-    (property "Intersheet References" "${INTERSHEET_REFS}" (id 0) (at 68.816 50.7206 0)
+    (property "Intersheet References" "${INTERSHEET_REFS}" (id 0) (at 70.7512 50.8794 0)
       (effects (font (size 1.27 1.27)) (justify left) hide)
     )
   )
-  (global_label "INT" (shape input) (at 139.7 31.75 180) (fields_autoplaced)
+  (global_label "IO{SDI}" (shape input) (at 38.1 48.26 180) (fields_autoplaced)
     (effects (font (size 1.27 1.27)) (justify right))
-    (property "Intersheet References" "${INTERSHEET_REFS}" (id 0) (at 134.384 31.8294 0)
+    (property "Intersheet References" "${INTERSHEET_REFS}" (id 0) (at 28.974 48.1806 0)
+      (effects (font (size 1.27 1.27)) (justify right) hide)
+    )
+  )
+  (global_label "IO{7}" (shape input) (at 139.7 31.75 180) (fields_autoplaced)
+    (effects (font (size 1.27 1.27)) (justify right))
+    (property "Intersheet References" "${INTERSHEET_REFS}" (id 0) (at 132.4488 31.6706 0)
+      (effects (font (size 1.27 1.27)) (justify right) hide)
+    )
+  )
+  (global_label "IO{SDO}" (shape input) (at 38.1 50.8 180) (fields_autoplaced)
+    (effects (font (size 1.27 1.27)) (justify right))
+    (property "Intersheet References" "${INTERSHEET_REFS}" (id 0) (at 28.2483 50.7206 0)
+      (effects (font (size 1.27 1.27)) (justify right) hide)
+    )
+  )
+  (global_label "IO{SCK, CSB, SDI, SDO}" (shape input) (at 139.7 41.91 180) (fields_autoplaced)
+    (effects (font (size 1.27 1.27)) (justify right))
+    (property "Intersheet References" "${INTERSHEET_REFS}" (id 0) (at 114.5479 41.8306 0)
+      (effects (font (size 1.27 1.27)) (justify right) hide)
+    )
+  )
+  (global_label "IO{SCK}" (shape input) (at 38.1 53.34 180) (fields_autoplaced)
+    (effects (font (size 1.27 1.27)) (justify right))
+    (property "Intersheet References" "${INTERSHEET_REFS}" (id 0) (at 28.3088 53.2606 0)
       (effects (font (size 1.27 1.27)) (justify right) hide)
     )
@@
       (effects (font (size 1.27 1.27)) (justify left))
     )
-    (property "Footprint" "" (id 2) (at 64.4652 40.64 0)
+    (property "Footprint" "Capacitor_SMD:C_0805_2012Metric" (id 2) (at 64.4652 40.64 0)
       (effects (font (size 1.27 1.27)) hide)
     )
@@
       (effects (font (size 1.27 1.27)) (justify left))
     )
-    (property "Footprint" "" (id 2) (at 35.2552 38.1 0)
+    (property "Footprint" "Capacitor_SMD:C_0805_2012Metric" (id 2) (at 35.2552 38.1 0)
       (effects (font (size 1.27 1.27)) hide)
     )
@@
     )
     (path "/d9abdac4-cfd8-4e19-8a5d-5e44f8b1424b"
-      (reference "C3") (unit 1) (value "1uF") (footprint "")
+      (reference "C3") (unit 1) (value "1uF") (footprint "Capacitor_SMD:C_0805_2012Metric")
     )
     (path "/d2d1c40e-f107-485d-abbe-8b041e6cd175"
-      (reference "C4") (unit 1) (value "0.1uF") (footprint "")
+      (reference "C4") (unit 1) (value "0.1uF") (footprint "Capacitor_SMD:C_0805_2012Metric")
     )
     (path "/7dba8d67-81e9-4f8d-bb03-bcf60266c722"

Commit message: Revised PCB and Sheet
Parts:
- added D1: LED, LED_SMD:LED_1812_4532Metric_Pad1.30x3.40mm_HandSolder, symbol Device:LED
- added R1: 200Ω, Resistor_SMD:R_0805_2012Metric, symbol Device:R
Connections:
- net +3V3 is gone; now on net +3.3V: C3.1, C4.1, U1.1 (Vdd_I/O), U1.6 (Vs)
- net +3.3V: now also R1.1
- net GND: now also D1.1 (K)
- net IO{7} renamed IO7
- net IO{CSB} renamed IO.CSB
- net IO{SCK} renamed IO.SCK
- net IO{SDI} renamed IO.SDO
- net IO{SDO} renamed IO.SDI
- new net: D1.2 (A), R1.2
Other:
- added sheet Accelerometer (accelerometer.kicad_sch)

Commit message: Finished shield design
Parts:
- removed C1, C3, C5: 1uF, Capacitor_SMD:C_0805_2012Metric, symbol Device:C
- removed C2, C6: 100 nF, Capacitor_SMD:C_0805_2012Metric, symbol Device:C
- removed C4: 0.1uF, Capacitor_SMD:C_0805_2012Metric, symbol Device:C
- removed D1: LED, LED_SMD:LED_1812_4532Metric_Pad1.30x3.40mm_HandSolder, symbol Device:LED
- removed R1: 200Ω, Resistor_SMD:R_0805_2012Metric, symbol Device:R
- removed U1: ADXL343, Package_LGA:LGA-14_3x5mm_P0.8mm_LayoutBorder1x6y, symbol Sensor_Motion:ADXL343
- removed U2: AZ1117, Package_TO_SOT_SMD:SOT-223-3_TabPin2, symbol Regulator_Linear:AZ1117-3.3
Connections:
- no-connect marks 6 -> 3
Other:
- sheet Accelerometer ports: added IO{7}, IO{SCK, CSB, SDO, SDI}; removed none
