File: FPGA_Pinout.kicad_sch (KiCad schematic)
At the start: 9 parts, among them J1 Conn_01x04_Male, J2 Conn_01x06_Male, J3 Conn_01x06_Male, J4 Conn_01x04_Male, J5 Conn_01x01_Male, J6 Conn_01x06_Male, J7 Conn_01x15_Male, J8 Conn_01x15_Male, J9 Conn_01x02_Male

Commit message: Finished shield design
Parts:
- renumbered J4 to J1, J5 to J2, J6 to J3, J1 to J4, J9 to J5, J2 to J6, J3 to J7, J7 to J8, J8 to J9
Changed lines of the file:
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@@
   (symbol (lib_id "power:GND") (at 123.19 128.27 0) (unit 1)
     (in_bom yes) (on_board yes) (fields_autoplaced)
-    (property "Reference" "#PWR010" (id 0) (at 123.19 134.62 0)
+    (property "Reference" "#PWR015" (id 0) (at 123.19 134.62 0)
       (effects (font (size 1.27 1.27)) hide)
     )
@@
   (symbol (lib_id "Connector:Conn_01x06_Male") (at 93.98 87.63 0) (unit 1)
     (in_bom yes) (on_board yes) (fields_autoplaced)
-    (property "Reference" "J3" (id 0) (at 94.615 77.47 0))
+    (property "Reference" "J7" (id 0) (at 94.615 77.47 0))
     (property "Value" "Conn_01x06_Male" (id 1) (at 94.615 80.01 0))
     (property "Footprint" "Connector_PinHeader_2.00mm:PinHeader_1x06_P2.00mm_Vertical" (id 2) (at 93.98 87.63 0)
@@
   (symbol (lib_id "power:GND") (at 52.07 97.79 0) (unit 1)
     (in_bom yes) (on_board yes) (fields_autoplaced)
-    (property "Reference" "#PWR07" (id 0) (at 52.07 104.14 0)
+    (property "Reference" "#PWR02" (id 0) (at 52.07 104.14 0)
       (effects (font (size 1.27 1.27)) hide)
     )
@@
   (symbol (lib_id "Connector:Conn_01x15_Male") (at 119.38 143.51 180) (unit 1)
     (in_bom yes) (on_board yes) (fields_autoplaced)
-    (property "Reference" "J8" (id 0) (at 118.745 167.005 0))
+    (property "Reference" "J9" (id 0) (at 118.745 167.005 0))
     (property "Value" "Conn_01x15_Male" (id 1) (at 118.745 164.465 0))
     (property "Footprint" "Connector_PinHeader_2.00mm:PinHeader_1x15_P2.00mm_Vertical" (id 2) (at 119.38 143.51 0)
@@
   (symbol (lib_id "power:+1V8") (at 52.07 133.35 270) (unit 1)
     (in_bom yes) (on_board yes) (fields_autoplaced)
-    (property "Reference" "#PWR011" (id 0) (at 48.26 133.35 0)
+    (property "Reference" "#PWR03" (id 0) (at 48.26 133.35 0)
       (effects (font (size 1.27 1.27)) hide)
     )
@@
   (symbol (lib_id "Connector:Conn_01x06_Male") (at 40.64 137.16 0) (unit 1)
     (in_bom yes) (on_board yes) (fields_autoplaced)
-    (property "Reference" "J6" (id 0) (at 41.275 127 0))
+    (property "Reference" "J3" (id 0) (at 41.275 127 0))
     (property "Value" "Conn_01x06_Male" (id 1) (at 41.275 129.54 0))
     (property "Footprint" "Connector_PinHeader_2.00mm:PinHeader_1x06_P2.00mm_Vertical" (id 2) (at 40.64 137.16 0)
@@
   (symbol (lib_id "Connector:Conn_01x04_Male") (at 40.64 88.9 0) (unit 1)
     (in_bom yes) (on_board yes) (fields_autoplaced)
-    (property "Reference" "J4" (id 0) (at 41.275 81.28 0))
+    (property "Reference" "J1" (id 0) (at 41.275 81.28 0))
     (property "Value" "Conn_01x04_Male" (id 1) (at 41.275 83.82 0))
     (property "Footprint" "Connector_PinHeader_2.00mm:PinHeader_1x04_P2.00mm_Vertical" (id 2) (at 40.64 88.9 0)
@@
   (symbol (lib_id "Connector:Conn_01x04_Male") (at 41.275 45.085 0) (unit 1)
     (in_bom yes) (on_board yes) (fields_autoplaced)
-    (property "Reference" "J1" (id 0) (at 41.91 37.465 0))
+    (property "Reference" "J4" (id 0) (at 41.91 37.465 0))
     (property "Value" "Conn_01x04_Male" (id 1) (at 41.91 40.005 0))
     (property "Footprint" "Connector_PinHeader_2.00mm:PinHeader_1x04_P2.00mm_Vertical" (id 2) (at 41.275 45.085 0)
@@
   (symbol (lib_id "power:+5V") (at 109.22 125.73 0) (unit 1)
     (in_bom yes) (on_board yes) (fields_autoplaced)
-    (property "Reference" "#PWR09" (id 0) (at 109.22 129.54 0)
+    (property "Reference" "#PWR014" (id 0) (at 109.22 129.54 0)
       (effects (font (size 1.27 1.27)) hide)
     )
@@
   (symbol (lib_id "Connector:Conn_01x02_Male") (at 43.18 167.64 0) (unit 1)
     (in_bom yes) (on_board yes) (fields_autoplaced)
-    (property "Reference" "J9" (id 0) (at 43.815 162.56 0))
+    (property "Reference" "J5" (id 0) (at 43.815 162.56 0))
     (property "Value" "Conn_01x02_Male" (id 1) (at 43.815 165.1 0))
     (property "Footprint" "Connector_PinHeader_2.00mm:PinHeader_1x02_P2.00mm_Vertical" (id 2) (at 43.18 167.64 0)
@@
   (symbol (lib_id "Connector:Conn_01x01_Male") (at 40.64 123.19 0) (unit 1)
     (in_bom yes) (on_board yes) (fields_autoplaced)
-    (property "Reference" "J5" (id 0) (at 41.275 118.11 0))
+    (property "Reference" "J2" (id 0) (at 41.275 118.11 0))
     (property "Value" "Conn_01x01_Male" (id 1) (at 41.275 120.65 0))
     (property "Footprint" "Connector_PinHeader_2.00mm:PinHeader_1x01_P2.00mm_Vertical" (id 2) (at 40.64 123.19 0)
@@
   (symbol (lib_id "power:+5V") (at 105.41 36.83 0) (unit 1)
     (in_bom yes) (on_board yes) (fields_autoplaced)
-    (property "Reference" "#PWR01" (id 0) (at 105.41 40.64 0)
+    (property "Reference" "#PWR010" (id 0) (at 105.41 40.64 0)
       (effects (font (size 1.27 1.27)) hide)
     )
@@
   (symbol (lib_id "power:+5V") (at 52.705 38.735 0) (unit 1)
     (in_bom yes) (on_board yes) (fields_autoplaced)
-    (property "Reference" "#PWR02" (id 0) (at 52.705 42.545 0)
+    (property "Reference" "#PWR06" (id 0) (at 52.705 42.545 0)
       (effects (font (size 1.27 1.27)) hide)
     )
@@
   (symbol (lib_id "power:GND") (at 52.07 142.24 0) (unit 1)
     (in_bom yes) (on_board yes) (fields_autoplaced)
-    (property "Reference" "#PWR017" (id 0) (at 52.07 148.59 0)
+    (property "Reference" "#PWR05" (id 0) (at 52.07 148.59 0)
       (effects (font (size 1.27 1.27)) hide)
     )
@@
   (symbol (lib_id "power:GND") (at 190.5 139.7 0) (unit 1)
     (in_bom yes) (on_board yes) (fields_autoplaced)
-    (property "Reference" "#PWR013" (id 0) (at 190.5 146.05 0)
+    (property "Reference" "#PWR016" (id 0) (at 190.5 146.05 0)
       (effects (font (size 1.27 1.27)) hide)
     )
@@
   (symbol (lib_id "power:GND") (at 53.34 171.45 0) (unit 1)
     (in_bom yes) (on_board yes) (fields_autoplaced)
-    (property "Reference" "#PWR019" (id 0) (at 53.34 177.8 0)
+    (property "Reference" "#PWR09" (id 0) (at 53.34 177.8 0)
       (effects (font (size 1.27 1.27)) hide)
     )
@@
   (symbol (lib_id "Connector:Conn_01x06_Male") (at 93.98 45.72 0) (unit 1)
     (in_bom yes) (on_board yes) (fields_autoplaced)
-    (property "Reference" "J2" (id 0) (at 94.615 35.56 0))
+    (property "Reference" "J6" (id 0) (at 94.615 35.56 0))
     (property "Value" "Conn_01x06_Male" (id 1) (at 94.615 38.1 0))
     (property "Footprint" "Connector_PinHeader_2.00mm:PinHeader_1x06_P2.00mm_Vertical" (id 2) (at 93.98 45.72 0)
@@
   (symbol (lib_id "power:+5V") (at 224.79 139.7 180) (unit 1)
     (in_bom yes) (on_board yes) (fields_autoplaced)
-    (property "Reference" "#PWR016" (id 0) (at 224.79 135.89 0)
+    (property "Reference" "#PWR019" (id 0) (at 224.79 135.89 0)
       (effects (font (size 1.27 1.27)) hide)
     )
@@
   (symbol (lib_id "power:+3.3V") (at 52.07 138.43 270) (unit 1)
     (in_bom yes) (on_board yes) (fields_autoplaced)
-    (property "Reference" "#PWR012" (id 0) (at 48.26 138.43 0)
+    (property "Reference" "#PWR04" (id 0) (at 48.26 138.43 0)
       (effects (font (size 1.27 1.27)) hide)
     )
@@
   (symbol (lib_id "power:GND") (at 105.41 55.88 0) (unit 1)
     (in_bom yes) (on_board yes) (fields_autoplaced)
-    (property "Reference" "#PWR04" (id 0) (at 105.41 62.23 0)
+    (property "Reference" "#PWR011" (id 0) (at 105.41 62.23 0)
       (effects (font (size 1.27 1.27)) hide)
     )
@@
   (symbol (lib_id "power:GND") (at 52.705 53.975 0) (unit 1)
     (in_bom yes) (on_board yes) (fields_autoplaced)
-    (property "Reference" "#PWR03" (id 0) (at 52.705 60.325 0)
+    (property "Reference" "#PWR07" (id 0) (at 52.705 60.325 0)
       (effects (font (size 1.27 1.27)) hide)
     )
@@
   (symbol (lib_id "power:+5V") (at 53.34 166.37 0) (unit 1)
     (in_bom yes) (on_board yes) (fields_autoplaced)
-    (property "Reference" "#PWR018" (id 0) (at 53.34 170.18 0)
+    (property "Reference" "#PWR08" (id 0) (at 53.34 170.18 0)
       (effects (font (size 1.27 1.27)) hide)
     )
@@
   (symbol (lib_id "power:GND") (at 105.41 97.79 0) (unit 1)
     (in_bom yes) (on_board yes) (fields_autoplaced)
-    (property "Reference" "#PWR08" (id 0) (at 105.41 104.14 0)
+    (property "Reference" "#PWR013" (id 0) (at 105.41 104.14 0)
       (effects (font (size 1.27 1.27)) hide)
     )
@@
   (symbol (lib_id "power:+1V8") (at 213.36 139.7 180) (unit 1)
     (in_bom yes) (on_board yes) (fields_autoplaced)
-    (property "Reference" "#PWR015" (id 0) (at 213.36 135.89 0)
+    (property "Reference" "#PWR018" (id 0) (at 213.36 135.89 0)
       (effects (font (size 1.27 1.27)) hide)
     )
@@
   (symbol (lib_id "power:+3.3V") (at 105.41 78.74 0) (unit 1)
     (in_bom yes) (on_board yes) (fields_autoplaced)
-    (property "Reference" "#PWR05" (id 0) (at 105.41 82.55 0)
+    (property "Reference" "#PWR012" (id 0) (at 105.41 82.55 0)
       (effects (font (size 1.27 1.27)) hide)
     )
@@
   (symbol (lib_id "power:+5V") (at 52.07 82.55 0) (unit 1)
     (in_bom yes) (on_board yes) (fields_autoplaced)
-    (property "Reference" "#PWR06" (id 0) (at 52.07 86.36 0)
+    (property "Reference" "#PWR01" (id 0) (at 52.07 86.36 0)
       (effects (font (size 1.27 1.27)) hide)
     )
@@
   (symbol (lib_id "power:+3.3V") (at 201.93 139.7 180) (unit 1)
     (in_bom yes) (on_board yes) (fields_autoplaced)
-    (property "Reference" "#PWR014" (id 0) (at 201.93 135.89 0)
+    (property "Reference" "#PWR017" (id 0) (at 201.93 135.89 0)
       (effects (font (size 1.27 1.27)) hide)
     )
@@
   (symbol (lib_id "Connector:Conn_01x15_Male") (at 100.33 143.51 180) (unit 1)
     (in_bom yes) (on_board yes) (fields_autoplaced)
-    (property "Reference" "J7" (id 0) (at 99.695 167.005 0))
+    (property "Reference" "J8" (id 0) (at 99.695 167.005 0))
     (property "Value" "Conn_01x15_Male" (id 1) (at 99.695 164.465 0))
     (property "Footprint" "Connector_PinHeader_2.00mm:PinHeader_1x15_P2.00mm_Vertical" (id 2) (at 100.33 143.51 0)
