File: accelerometer.kicad_sch (KiCad schematic)
At the start: 10 parts

Commit message: Finished shield design
Parts:
- gave numbers to parts that had none: 10
Connections:
- net +3.3V: no longer C3.1, C4.1, R1.1, U1.1 (Vdd_I/O), U1.6 (Vs)
- new net +3V3: C3.1, C4.1, R1.1, U1.1 (Vdd_I/O), U1.6 (Vs)
Changed lines of the file:
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@@
-    (stroke (width 0) (type default) (color 0 0 0 0))
-  )
-  (wire (pts (xy 210.82 50.8) (xy 215.9 50.8))
     (stroke (width 0) (type default) (color 0 0 0 0))
   )
@@
     (stroke (width 0) (type default) (color 0 0 0 0))
   )
+  (bus (pts (xy 210.82 55.88) (xy 214.63 55.88))
+    (stroke (width 0) (type default) (color 0 0 0 0))
+  )
   (wire (pts (xy 78.74 121.92) (xy 78.74 125.73))
     (stroke (width 0) (type default) (color 0 0 0 0))
@@
     )
   )
-  (global_label "3.3V" (shape input) (at 55.88 46.99 90) (fields_autoplaced)
+  (global_label "IO7" (shape input) (at 91.44 67.31 0) (fields_autoplaced)
     (effects (font (size 1.27 1.27)) (justify left))
-    (property "Intersheet References" "${INTERSHEET_REFS}" (id 0) (at 55.8006 40.4645 90)
+    (property "Intersheet References" "${INTERSHEET_REFS}" (id 0) (at 96.9979 67.2306 0)
       (effects (font (size 1.27 1.27)) (justify left) hide)
     )
   )
-  (global_label "3.3V" (shape input) (at 130.81 73.66 180) (fields_autoplaced)
-    (effects (font (size 1.27 1.27)) (justify right))
-    (property "Intersheet References" "${INTERSHEET_REFS}" (id 0) (at 124.2845 73.7394 0)
-      (effects (font (size 1.27 1.27)) (justify right) hide)
-    )
-  )
-  (global_label "IO7" (shape input) (at 210.82 50.8 180) (fields_autoplaced)
-    (effects (font (size 1.27 1.27)) (justify right))
-    (property "Intersheet References" "${INTERSHEET_REFS}" (id 0) (at 205.2621 50.7206 0)
-      (effects (font (size 1.27 1.27)) (justify right) hide)
-    )
-  )
-  (global_label "3.3V" (shape input) (at 99.06 114.3 90) (fields_autoplaced)
+  (global_label "IO.SDI" (shape input) (at 66.04 67.31 180) (fields_autoplaced)
+    (effects (font (size 1.27 1.27)) (justify right))
+    (property "Intersheet References" "${INTERSHEET_REFS}" (id 0) (at 58.0026 67.2306 0)
+      (effects (font (size 1.27 1.27)) (justify right) hide)
+    )
+  )
+  (global_label "IO.CSB" (shape input) (at 66.04 72.39 180) (fields_autoplaced)
+    (effects (font (size 1.27 1.27)) (justify right))
+    (property "Intersheet References" "${INTERSHEET_REFS}" (id 0) (at 57.3374 72.3106 0)
+      (effects (font (size 1.27 1.27)) (justify right) hide)
+    )
+  )
+  (global_label "IO.SDO" (shape input) (at 66.04 64.77 180) (fields_autoplaced)
+    (effects (font (size 1.27 1.27)) (justify right))
+    (property "Intersheet References" "${INTERSHEET_REFS}" (id 0) (at 57.2769 64.6906 0)
+      (effects (font (size 1.27 1.27)) (justify right) hide)
+    )
+  )
+  (global_label "IO{7}" (shape input) (at 210.82 55.88 180) (fields_autoplaced)
+    (effects (font (size 1.27 1.27)) (justify right))
+    (property "Sayfalar Arası Referanslar" "${INTERSHEET_REFS}" (id 0) (at 203.5688 55.8006 0)
+      (effects (font (size 1.27 1.27)) (justify right) hide)
+    )
+  )
+  (global_label "IO.SCK" (shape input) (at 66.04 69.85 180) (fields_autoplaced)
+    (effects (font (size 1.27 1.27)) (justify right))
+    (property "Intersheet References" "${INTERSHEET_REFS}" (id 0) (at 57.3374 69.7706 0)
+      (effects (font (size 1.27 1.27)) (justify right) hide)
+    )
+  )
+  (hierarchical_label "IO{7}" (shape input) (at 214.63 55.88 0)
     (effects (font (size 1.27 1.27)) (justify left))
-    (property "Intersheet References" "${INTERSHEET_REFS}" (id 0) (at 98.9806 107.7745 90)
-      (effects (font (size 1.27 1.27)) (justify left) hide)
-    )
-  )
-  (hierarchical_label "INT" (shape input) (at 91.44 67.31 0)
-    (effects (font (size 1.27 1.27)) (justify left))
-  )
-  (hierarchical_label "IO.SDO" (shape input) (at 66.04 64.77 180)
-    (effects (font (size 1.27 1.27)) (justify right))
-  )
-  (hierarchical_label "INT" (shape input) (at 215.9 50.8 0)
-    (effects (font (size 1.27 1.27)) (justify left))
-  )
-  (hierarchical_label "IO.CSB" (shape input) (at 66.04 72.39 180)
-    (effects (font (size 1.27 1.27)) (justify right))
-  )
-  (hierarchical_label "IO.SCK" (shape input) (at 66.04 69.85 180)
-    (effects (font (size 1.27 1.27)) (justify right))
   )
   (hierarchical_label "IO{SCK, CSB, SDO, SDI}" (shape input) (at 215.9 45.72 0)
     (effects (font (size 1.27 1.27)) (justify left))
   )
-  (hierarchical_label "IO.SDI" (shape input) (at 66.04 67.31 180)
-    (effects (font (size 1.27 1.27)) (justify right))
-  )
   (symbol (lib_id "Device:C") (at 62.23 50.8 0) (unit 1)
     (in_bom yes) (on_board yes) (fields_autoplaced)
-    (property "Reference" "C?" (id 0) (at 66.04 49.5299 0)
+    (property "Reference" "C3" (id 0) (at 66.04 49.5299 0)
       (effects (font (size 1.27 1.27)) (justify left))
     )
@@
   (symbol (lib_name "+3.3V_1") (lib_id "power:+3.3V") (at 50.8 46.99 0) (unit 1)
     (in_bom yes) (on_board yes) (fields_autoplaced)
-    (property "Reference" "#PWR?" (id 0) (at 50.8 50.8 0)
+    (property "Reference" "#PWR021" (id 0) (at 50.8 50.8 0)
       (effects (font (size 1.27 1.27)) hide)
     )
@@
   (symbol (lib_id "Device:C") (at 104.14 119.38 0) (unit 1)
     (in_bom yes) (on_board yes)
-    (property "Reference" "C?" (id 0) (at 105.41 116.84 0)
+    (property "Reference" "C6" (id 0) (at 105.41 116.84 0)
       (effects (font (size 1.27 1.27)) (justify left))
     )
@@
   (symbol (lib_id "Sensor_Motion:ADXL343") (at 78.74 67.31 0) (unit 1)
     (in_bom yes) (on_board yes)
-    (property "Reference" "U?" (id 0) (at 93.98 60.7312 0)
+    (property "Reference" "U1" (id 0) (at 93.98 60.7312 0)
       (effects (font (size 1.27 1.27)) hide)
     )
@@
   (symbol (lib_id "power:GND") (at 78.74 128.27 0) (unit 1)
     (in_bom yes) (on_board yes)
-    (property "Reference" "#PWR?" (id 0) (at 78.74 134.62 0)
+    (property "Reference" "#PWR024" (id 0) (at 78.74 134.62 0)
       (effects (font (size 1.27 1.27)) hide)
     )
@@
   (symbol (lib_id "Device:R") (at 130.81 82.55 0) (unit 1)
     (in_bom yes) (on_board yes) (fields_autoplaced)
-    (property "Reference" "R?" (id 0) (at 133.35 81.2799 0)
+    (property "Reference" "R1" (id 0) (at 133.35 81.2799 0)
       (effects (font (size 1.27 1.27)) (justify left))
     )
@@
   (symbol (lib_id "Device:C") (at 93.98 119.38 0) (unit 1)
     (in_bom yes) (on_board yes)
-    (property "Reference" "C?" (id 0) (at 95.25 116.84 0)
+    (property "Reference" "C5" (id 0) (at 95.25 116.84 0)
       (effects (font (size 1.27 1.27)) (justify left))
     )
@@
   (symbol (lib_id "power:GND") (at 91.44 57.15 0) (unit 1)
     (in_bom yes) (on_board yes) (fields_autoplaced)
-    (property "Reference" "#PWR?" (id 0) (at 91.44 63.5 0)
+    (property "Reference" "#PWR025" (id 0) (at 91.44 63.5 0)
       (effects (font (size 1.27 1.27)) hide)
     )
@@
   (symbol (lib_name "+3.3V_2") (lib_id "power:+3.3V") (at 130.81 69.85 0) (unit 1)
     (in_bom yes) (on_board yes) (fields_autoplaced)
-    (property "Reference" "#PWR?" (id 0) (at 130.81 73.66 0)
+    (property "Reference" "#PWR027" (id 0) (at 130.81 73.66 0)
       (effects (font (size 1.27 1.27)) hide)
     )
@@
   (symbol (lib_id "power:GND") (at 78.74 80.01 0) (unit 1)
     (in_bom yes) (on_board yes) (fields_autoplaced)
-    (property "Reference" "#PWR?" (id 0) (at 78.74 86.36 0)
+    (property "Reference" "#PWR023" (id 0) (at 78.74 86.36 0)
       (effects (font (size 1.27 1.27)) hide)
     )
@@
   (symbol (lib_id "power:+5V") (at 46.99 114.3 0) (unit 1)
     (in_bom yes) (on_board yes)
-    (property "Reference" "#PWR?" (id 0) (at 46.99 118.11 0)
+    (property "Reference" "#PWR020" (id 0) (at 46.99 118.11 0)
       (effects (font (size 1.27 1.27)) hide)
     )
@@
   (symbol (lib_id "Device:C") (at 91.44 53.34 0) (unit 1)
     (in_bom yes) (on_board yes) (fields_autoplaced)
-    (property "Reference" "C?" (id 0) (at 95.25 52.0699 0)
+    (property "Reference" "C4" (id 0) (at 95.25 52.0699 0)
       (effects (font (size 1.27 1.27)) (justify left))
     )
@@
   (symbol (lib_id "power:GND") (at 130.81 101.6 0) (unit 1)
     (in_bom yes) (on_board yes) (fields_autoplaced)
-    (property "Reference" "#PWR?" (id 0) (at 130.81 107.95 0)
+    (property "Reference" "#PWR028" (id 0) (at 130.81 107.95 0)
       (effects (font (size 1.27 1.27)) hide)
     )
@@
   (symbol (lib_id "Device:C") (at 60.96 119.38 0) (unit 1)
     (in_bom yes) (on_board yes)
-    (property "Reference" "C?" (id 0) (at 62.23 116.84 0)
+    (property "Reference" "C2" (id 0) (at 62.23 116.84 0)
       (effects (font (size 1.27 1.27)) (justify left))
     )
@@
   (symbol (lib_id "Device:LED") (at 130.81 90.17 90) (unit 1)
     (in_bom yes) (on_board yes) (fields_autoplaced)
-    (property "Reference" "D?" (id 0) (at 134.62 90.4874 90)
+    (property "Reference" "D1" (id 0) (at 134.62 90.4874 90)
       (effects (font (size 1.27 1.27)) (justify right))
     )
@@
   (symbol (lib_id "Device:C") (at 50.8 119.38 0) (unit 1)
     (in_bom yes) (on_board yes)
-    (property "Reference" "C?" (id 0) (at 52.07 116.84 0)
+    (property "Reference" "C1" (id 0) (at 52.07 116.84 0)
       (effects (font (size 1.27 1.27)) (justify left))
     )
@@
   (symbol (lib_id "power:GND") (at 62.23 54.61 0) (unit 1)
     (in_bom yes) (on_board yes) (fields_autoplaced)
-    (property "Reference" "#PWR?" (id 0) (at 62.23 60.96 0)
+    (property "Reference" "#PWR022" (id 0) (at 62.23 60.96 0)
       (effects (font (size 1.27 1.27)) hide)
     )
@@
   (symbol (lib_id "power:+3.3V") (at 109.22 114.3 0) (unit 1)
     (in_bom yes) (on_board yes) (fields_autoplaced)
-    (property "Reference" "#PWR?" (id 0) (at 109.22 118.11 0)
+    (property "Reference" "#PWR026" (id 0) (at 109.22 118.11 0)
       (effects (font (size 1.27 1.27)) hide)
     )
@@
   (symbol (lib_id "Regulator_Linear:AZ1117-3.3") (at 78.74 114.3 0) (unit 1)
     (in_bom yes) (on_board yes) (fields_autoplaced)
-    (property "Reference" "U?" (id 0) (at 78.74 106.68 0))
+    (property "Reference" "U2" (id 0) (at 78.74 106.68 0))
     (property "Value" "AZ1117" (id 1) (at 78.74 109.22 0))
     (property "Footprint" "Package_TO_SOT_SMD:SOT-223-3_TabPin2" (id 2) (at 78.74 107.95 0)
